File: electronics/PC_driver/PC_driver.kicad_pcb (KiCad board)
At the start: 2 copper layers, 77.5 x 64.8 mm, 18 parts, among them J1 Analog PC INP, J2 Analog OUT, J3 TTL INP, J4 Jack-DC, SW1 SW_SPDT

Commit message: finished schmatics and footprint association
Parts:
- removed AGD1: AGD419BN2, Housings_DIP:DIP-8_W7.62mm
- removed CA1: CA3240, Housings_DIP:DIP-8_W10.16mm
- removed LM101: LM10CLN, Housings_DIP:DIP-8_W10.16mm
- added C3: 100nF, Capacitor_THT:C_Disc_D5.0mm_W2.5mm_P2.50mm, F.Cu at (202.4, 98.9)
- added D2: switch_led, LED_THT:LED_D5.0mm_Clear, F.Cu at (226.4, 86.6)
- added P1: USB_C_Plug_USB2.0, Connector_USB:USB_C_Receptacle_GCT_USB4085, F.Cu at (215.2, 90.6)
- added R7: 3k6, Resistor_THT:R_Axial_DIN0309_L9.0mm_D3.2mm_P15.24mm_Horizontal, F.Cu at (163.7, 94.5)
- added U1: LM10CLN, Package_DIP:DIP-8_W7.62mm, F.Cu at (214.0, 79.3)
- added U2: CA3240AE, Package_DIP:DIP-8_W7.62mm, F.Cu at (229.8, 73.2)
- added U3: ADG419BN, Package_DIP:DIP-8_W7.62mm, F.Cu at (229.6, 61.4)
- C1: footprint Capacitors_THT:C_Rect_L10.3mm_W4.5mm_P7.50mm_MKS4 -> Capacitor_THT:C_Disc_D5.0mm_W2.5mm_P2.50mm
- C2: footprint Capacitors_THT:C_Rect_L13.0mm_W4.0mm_P10.00mm_FKS3_FKP3_MKS4 -> Capacitor_THT:C_Disc_D5.0mm_W2.5mm_P2.50mm
- D1: value LED -> potent_led; footprint LEDs:LED_PLCC-2 -> LED_THT:LED_D5.0mm_Clear
- J1: value Analog PC INP -> Analog_Input (0-5V); footprint Connectors:BNC -> Connector_Coaxial:BNC_Amphenol_B6252HB-NPP3G-50_Horizontal
- J2: value Analog OUT -> add_resist_jumper; footprint Connectors:BNC -> Connector_PinHeader_2.54mm:PinHeader_1x03_P2.54mm_Vertical
- J3: value TTL INP -> Analog_out (0to5V); footprint Connectors:BNC -> Connector_Coaxial:BNC_Amphenol_B6252HB-NPP3G-50_Horizontal
- J4: value Jack-DC -> TTL_input (blanking); footprint Connectors:BARREL_JACK -> Connector_Coaxial:BNC_Amphenol_B6252HB-NPP3G-50_Horizontal
- R1, R2, R3, R4, R5, R6: footprint Resistors_THT:R_Axial_DIN0207_L6.3mm_D2.5mm_P10.16mm_Horizontal -> Resistor_THT:R_Axial_DIN0309_L9.0mm_D3.2mm_P12.70mm_Horizontal
- RV1: value POT -> laser_int 5k; footprint Potentiometers:Potentiometer_WirePads -> Potentiometer_THT:Potentiometer_ACP_CA14-H5_Horizontal
- SW1: footprint Buttons_Switches_SMD:SW_SPDT_CK-JS102011SAQN -> Button_Switch_THT:SW_E-Switch_EG1224_SPDT_Angled
- moved RV1 91.3 mm to (240.9, 86.6), turned to 0 degrees
- moved R4 82.4 mm to (229.6, 57.0)
- moved D1 80.3 mm to (241.5, 72.8)
- moved J4 77.6 mm to (202.4, 64.4), turned to 0 degrees
- moved J2 76.1 mm to (241.2, 61.7), turned to 0 degrees
- moved R3 75.7 mm to (213.9, 74.9)
- moved SW1 66.2 mm to (216.2, 58.2), turned to 0 degrees
- moved C2 46.8 mm to (226.0, 92.4)
- moved R2 39.2 mm to (197.9, 94.5)
- moved R5 37.8 mm to (179.5, 99.3)
- moved R6 25.7 mm to (182.1, 94.5)
- moved R1 22.4 mm to (163.7, 99.3)
- moved J1 19.8 mm to (164.6, 65.3), turned to 0 degrees
- moved C1 13.9 mm to (195.8, 98.9)
- moved J3 0.76 mm to (184.7, 65.0), turned to 0 degrees
Connections:
- C1 pad 1: +5V -> pin2
- C1 pad 2: w2 -> internal_signal
- C2 pad 1: GND -> internal_signal
- C2 pad 2: +5V -> GND
- D1 pad 2: +5V -> internal_signal
- J1 pad 1: Net-(J1-Pad1) -> analog_input
- J1 pad 2: Net-(J1-Pad2) -> GND
- J2 pad 1: Net-(CA1-Pad6) -> Net-(J2-Pad1)
- J3 pad 1: Net-(AGD1-Pad6) -> Net-(J3-Pad1)
- J4 pad 1: +5V -> Net-(J4-Pad1)
- R1 pad 1: Net-(J1-Pad1) -> GND
- R1 pad 2: GND -> analog_input
- R2 pad 1: w2 -> internal_signal
- R2 pad 2: +5V -> pin2
- R3 pad 1: w2 -> pin2
- R3 pad 2: Net-(LM101-Pad4) -> GND
- R4 pad 1: Net-(CA1-Pad5) -> signal_pos_blank
- R4 pad 2: D -> Net-(J2-Pad1)
- R5 pad 1: GND -> Net-(D1-Pad1)
- R5 pad 2: Net-(D1-Pad1) -> GND
- R6 pad 1: Net-(AGD1-Pad6) -> Net-(J4-Pad1)
- RV1 pad 3: Net-(LM101-Pad4) -> GND
- SW1 pad 1: +5V -> internal_signal
- SW1 pad 3: Net-(J1-Pad1) -> analog_input
Routing:
- net Net-(J1-Pad1): track 127.1 -> 0.00 mm
- net Net-(CA1-Pad6): track 118.7 -> 0.00 mm
- net Net-(AGD1-Pad6): track 102.2 -> 0.00 mm
- net w2: track 82.2 -> 0.00 mm
- net Net-(RV1-Pad1): track 69.6 -> 0.00 mm
- net Net-(LM101-Pad4): track 66.2 -> 0.00 mm, vias 2 -> 0
- net D: track 66.1 -> 0.00 mm
- net Net-(RV1-Pad2): track 63.1 -> 0.00 mm
- net Net-(CA1-Pad5): track 61.4 -> 0.00 mm
- net Net-(SW1-Pad2): track 54.0 -> 0.00 mm
- net Net-(D1-Pad1): track 26.8 -> 0.00 mm, vias 2 -> 0
- net S2: track 11.4 -> 0.00 mm
- removed copper zone on F.Cu, net +5V
- removed copper zone on B.Cu, net GND
Other:
- board outline removed

Commit message: finish part placement, wiring and plotting
Parts:
- added REF**: KiCad-Logo2_5mm_SilkScreen, Symbol:KiCad-Logo2_5mm_SilkScreen, F.Cu at (162.5, 98.8)
- added REF**: OSHW-Logo2_7.3x6mm_SilkScreen, Symbol:OSHW-Logo2_7.3x6mm_SilkScreen, F.Cu at (150.9, 99.3)
- added REF**: MountingHole_3.2mm_M3_DIN965, MountingHole:MountingHole_3.2mm_M3_DIN965, F.Cu at (97.0, 53.0)
- added REF**: MountingHole_3.2mm_M3_DIN965, MountingHole:MountingHole_3.2mm_M3_DIN965, F.Cu at (185.0, 53.0)
- added REF**: MountingHole_3.2mm_M3_DIN965, MountingHole:MountingHole_3.2mm_M3_DIN965, F.Cu at (185.0, 98.0)
- added REF**: MountingHole_3.2mm_M3_DIN965, MountingHole:MountingHole_3.2mm_M3_DIN965, F.Cu at (97.0, 98.0)
- R3: renamed from R4; value 60 -> 3k6
- R4: renamed from R5; value 3k6 -> 60
- R7: footprint Resistor_THT:R_Axial_DIN0309_L9.0mm_D3.2mm_P15.24mm_Horizontal -> Resistor_THT:R_Axial_DIN0309_L9.0mm_D3.2mm_P12.70mm_Horizontal
- moved J2 135.2 mm to (108.0, 85.0), turned to 90 degrees
- moved U2 123.9 mm to (106.0, 70.0)
- moved SW1 114.4 mm to (109.0, 98.0)
- moved P1 108.9 mm to (113.0, 53.0), turned to 180 degrees
- moved D2 101.1 mm to (126.0, 98.0)
- moved U3 95.0 mm to (135.0, 70.0)
- moved C2 80.8 mm to (119.0, 74.0), turned to 90 degrees
- moved R5 77.0 mm to (126.0, 67.0), turned to 270 degrees
- moved R3 75.2 mm to (163.0, 92.0), turned to 180 degrees
- moved D1 73.9 mm to (172.0, 98.0)
- moved R1 69.8 mm to (104.0, 63.0)
- moved R2 64.9 mm to (150.0, 86.0)
- moved C1 64.3 mm to (165.0, 72.0), turned to 270 degrees
- moved U1 62.7 mm to (152.0, 70.0)
- moved RV1 62.4 mm to (181.0, 69.0)
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- renumbered C2 to C1, C1 to C2, R3 to R2, R2 to R5
Connections:
- C1 pad 1: internal_signal -> GND
- C1 pad 2: GND -> +5V
- C3 pad 1: GND -> +5V
- C3 pad 2: internal_signal -> GND
- D1 pad 2: internal_signal -> +5V
- D2 pad 2: internal_signal -> +5V
- J3 pad 2: Net-(J3-Pad2) -> GND
- P1 pad A4: internal_signal -> +5V
- P1 pad A9: internal_signal -> +5V
- P1 pad B4: internal_signal -> +5V
- P1 pad B9: internal_signal -> +5V
- R3 pad 1: signal_pos_blank -> Net-(D1-Pad1)
- R3 pad 2: Net-(J2-Pad1) -> GND
- R4 pad 1: Net-(D1-Pad1) -> signal_pos_blank
- R4 pad 2: GND -> Net-(J2-Pad1)
- U1 pad 7: internal_signal -> +5V
- U2 pad 8: internal_signal -> +5V
- U3 pad 4: internal_signal -> +5V
- U3 pad 5: internal_signal -> +5V
Routing:
- net internal_signal: track 0.00 -> 76.5 mm
- net pin2: track 0.00 -> 54.3 mm
- net analog_input: track 0.00 -> 49.4 mm, vias 0 -> 1
- net Net-(J4-Pad1): track 0.00 -> 44.6 mm
- net Net-(J3-Pad1): track 0.00 -> 44.1 mm
- net signal_pre_blank: track 0.00 -> 43.3 mm, vias 0 -> 2
- net Net-(RV1-Pad2): track 0.00 -> 40.2 mm
- net signal_pos_blank: track 0.00 -> 36.0 mm
- net Net-(RV1-Pad1): track 0.00 -> 29.4 mm
- net Net-(SW1-Pad2): track 0.00 -> 26.9 mm
- net Net-(D2-Pad1): track 0.00 -> 11.7 mm
- net Net-(D1-Pad1): track 0.00 -> 11.5 mm
- net +5V: track 0.00 -> 8.97 mm
- net Net-(J2-Pad2): track 0.00 -> 8.66 mm
- net GND: track 0.00 -> 8.28 mm
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- added copper zone on F.Cu, net +5V
- added copper zone on B.Cu, net GND
Other:
- board outline added: 98 x 57 mm
- net class thick added: clearance 0.3, trace_width 0.5, via_dia 0.65, via_drill 0.45
- board text added: "Pockel cell driver V. 0.1 CERN OHL V2 Design by R. Berndt @ HIH Tuebingen KiCad "translation" by F. Janiack & A. Maia Chagas 2020-06-02"

Commit message: correct misspelling
Other:
- board text added: "Pockel cell driver V. 0.1 CERN OHL V2 Design by R. Berndt @ HIH Tuebingen KiCad "translation" by F. Janiak & A. Maia Chagas 2020-06-02"
- board text removed: "Pockel cell driver V. 0.1 CERN OHL V2 Design by R. Berndt @ HIH Tuebingen KiCad "translation" by F. Janiack & A. Maia Chagas 2020-06-02"
